File: PCB/KiCAD/LED-Dimmer.kicad_sch (KiCad schematic)
At the start: 9 parts, among them Q1 BC547, U1 NE555D

Commit message: Update title
Other:
- title: Learn PCB Design -> Learn PCB Design-LED Dimmer
Changed lines of the file:
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@@
 	(paper "A4")
 	(title_block
-		(title "Learn PCB Design")
+		(title "Learn PCB Design-LED Dimmer")
 		(date "2025-11-19")
 		(rev "1.0.0")
